File: Hardware/PCB/pmf/pots.kicad_sch (KiCad schematic)
At the start: 39 parts, among them U3 TL074, U4 TL072

Commit message: Return to smaller trimmer values; make core schematic clearer; restore munged footprints
Parts:
- C14: footprint AO_tht:C_Disc_D3.0mm_W1.6mm_P2.50mm -> AO_tht:C_Rect_L7.2mm_W2.5mm_P5.00mm_FKS2_FKP2_MKS2_MKP2
- RV11, RV5: footprint AO_tht:Potentiometer_Bourns_3296W_Vertical_standard -> pmf:Potentiometer_Bourns_3296X_Horizontal
Changed lines of the file:
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@@
       (effects (font (size 1.27 1.27)))
     )
-    (property "Footprint" "AO_tht:Potentiometer_Bourns_3296W_Vertical_standard" (at 120.65 90.17 0)
+    (property "Footprint" "pmf:Potentiometer_Bourns_3296X_Horizontal" (at 120.65 90.17 0)
       (effects (font (size 1.27 1.27)) hide)
     )
@@
       (effects (font (size 1.27 1.27)) (justify left))
     )
-    (property "Footprint" "AO_tht:C_Disc_D3.0mm_W1.6mm_P2.50mm" (at 145.7452 99.06 0)
+    (property "Footprint" "AO_tht:C_Rect_L7.2mm_W2.5mm_P5.00mm_FKS2_FKP2_MKS2_MKP2" (at 145.7452 99.06 0)
       (effects (font (size 1.27 1.27)) hide)
     )
@@
       (effects (font (size 1.27 1.27)) (justify right))
     )
-    (property "Footprint" "AO_tht:Potentiometer_Bourns_3296W_Vertical_standard" (at 63.5 64.77 0)
-      (effects (font (size 1.27 1.27)) hide)
-    )
+    (property "Footprint" "pmf:Potentiometer_Bourns_3296X_Horizontal" (at 63.5 64.77 0)
+      (effects (font (size 1.27 1.27)) hide)
+    )

Commit message: Hardware symbols test
Parts:
- C14: footprint AO_tht:C_Rect_L7.2mm_W2.5mm_P5.00mm_FKS2_FKP2_MKS2_MKP2 -> AO_tht:C_Disc_D3.0mm_W1.6mm_P2.50mm
- RV11, RV5: footprint pmf:Potentiometer_Bourns_3296X_Horizontal -> AO_tht:Potentiometer_Bourns_3296W_Vertical_standard
Changed lines of the file:
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@@
       (effects (font (size 1.27 1.27)))
     )
-    (property "Footprint" "pmf:Potentiometer_Bourns_3296X_Horizontal" (at 120.65 90.17 0)
+    (property "Footprint" "AO_tht:Potentiometer_Bourns_3296W_Vertical_standard" (at 120.65 90.17 0)
       (effects (font (size 1.27 1.27)) hide)
     )
@@
       (effects (font (size 1.27 1.27)) (justify left))
     )
-    (property "Footprint" "AO_tht:C_Rect_L7.2mm_W2.5mm_P5.00mm_FKS2_FKP2_MKS2_MKP2" (at 145.7452 99.06 0)
+    (property "Footprint" "AO_tht:C_Disc_D3.0mm_W1.6mm_P2.50mm" (at 145.7452 99.06 0)
       (effects (font (size 1.27 1.27)) hide)
     )
@@
       (effects (font (size 1.27 1.27)) (justify right))
     )
-    (property "Footprint" "pmf:Potentiometer_Bourns_3296X_Horizontal" (at 63.5 64.77 0)
-      (effects (font (size 1.27 1.27)) hide)
-    )
+    (property "Footprint" "AO_tht:Potentiometer_Bourns_3296W_Vertical_standard" (at 63.5 64.77 0)
+      (effects (font (size 1.27 1.27)) hide)
+    )
