File: Hardware/pmf_panel/pmf_panel.kicad_pcb (KiCad board)
At the start: 2 copper layers, 100 x 200 mm, 15 parts

Commit message: panel
Parts:
- removed H12: Trimmer_Hole, Kosmo_panel:Kosmo_Trimmer_Pot_Hole
- removed H13: Led_Hole, Kosmo_panel:Kosmo_LED_Hole
- added GRAF1: Holes, pmf_panel:pmf_panel_holes, F.Cu at (116.1, 157.6)
- added GRAF2: Art, pmf_panel:pmf_panel_art, F.Cu at (116.1, 157.6)
- added H15: Pot_Hole, Kosmo_panel:Kosmo_Pot_Hole, F.Cu at (91.1, 177.6)
- added H16: Pot_Hole, Kosmo_panel:Kosmo_Pot_Hole, F.Cu at (91.1, 137.6)
- H11, H14: value Panel -> Mounting_Holes
- H7, H8: value Jack_Hole -> Pot_Hole; footprint Kosmo_panel:Kosmo_Jack_Hole -> Kosmo_panel:Kosmo_Pot_Hole
- H9: value Switch_Hole -> Rotary_Switch_Hole; footprint Kosmo_panel:Kosmo_Switch_Hole -> Kosmo_panel:Kosmo_Jack_Hole
- moved H7 130.9 mm to (91.1, 92.6)
- moved H9 78.1 mm to (141.1, 137.6)
- moved H8 56.4 mm to (141.1, 177.6)
- moved H5 35.4 mm to (153.6, 232.6)
- moved H10 8.74 mm to (141.1, 92.6)
Other:
- board text added: "Panel design by Rich Holmes CC0 1.0 May 2023 JLCJLCJLCJLC"
- board text removed: "Panel design by Rich Holmes CC0 1.0 ?? 2021 JLCJLCJLCJLC"
