File: Hardware/pmf_panel/pmf_panel.kicad_sch (KiCad schematic)
At the start: 17 parts

Commit message: panel
Parts:
- removed H12: Trimmer_Hole, Kosmo_panel:Kosmo_Trimmer_Pot_Hole, symbol Kosmo:Trimmer_Hole
- removed H13: Led_Hole, Kosmo_panel:Kosmo_LED_Hole, symbol Kosmo:Led_Hole
- removed H7, H8: Jack_Hole, Kosmo_panel:Kosmo_Jack_Hole, symbol Kosmo:Jack_Hole
- removed H9: Switch_Hole, Kosmo_panel:Kosmo_Switch_Hole, symbol Kosmo:Switch_Hole
- added H15, H16, H7, H8: Pot_Hole, Kosmo_panel:Kosmo_Pot_Hole, symbol Kosmo:Pot_Hole
- added H9: Rotary_Switch_Hole, Kosmo_panel:Kosmo_Jack_Hole, symbol Kosmo:Jack_Hole
- GRAF1: footprint (none) -> pmf_panel:pmf_panel_holes
- GRAF2: footprint (none) -> pmf_panel:pmf_panel_art
- H11, H14: footprint Kosmo_panel:Kosmo_Panel_Dual_Mounting_Holes -> Kosmo_panel:Kosmo_Panel_Dual_Slotted_Mounting_Holes
Connections:
- net GND: now also H15.1, H16.1, H7.1, H8.1, H9.1
Other:
- moved on the sheet: H10
